File: keezer.kicad_pcb (KiCad board)
At the start: 2 copper layers, 69.1 x 53.8 mm, 58 parts, among them J1 Barrel_Jack, J10 REF, J11 Display, J12 Mode, J13 Tare, J14 Rocker, J15 Temp VCC, J2 Relay, J3 Fan, J4 Temp 1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

Commit message: Logo. Finally.
Parts:
- added G***: LOGO, keezer:CRABBS, F.Cu at (99.9, 107.1)
